Commit message: checked differential drive model

File: mpc_ros_description/urdf/diff/differential_bot.gazebo.xacro (robot description, xacro)
@@ -64,5 +64,5 @@
   </gazebo>
   <gazebo>
-    <plugin name="servingbot_controller" filename="libgazebo_ros_diff_drive.so">
+    <plugin name="differential_controller" filename="libgazebo_ros_diff_drive.so">
       <commandTopic>cmd_vel</commandTopic>
       <odometryTopic>odom</odometryTopic>

File: mpc_ros_description/urdf/diff/differential_bot.urdf.xacro (robot description, xacro)
@@ -1,6 +1,6 @@
 <?xml version="1.0" ?>
 <robot name="differential_bot" xmlns:xacro="http://ros.org/wiki/xacro">
-  <xacro:include filename="$(find mpc_model_description)/urdf/common/common_properties.xacro"/>
-  <xacro:include filename="$(find mpc_model_description)/urdf/diff/differential_bot.gazebo.xacro"/>
+  <xacro:include filename="$(find mpc_ros_description)/urdf/common/common_properties.xacro"/>
+  <xacro:include filename="$(find mpc_ros_description)/urdf/diff/differential_bot.gazebo.xacro"/>
 <!-- base -->
 <link name="base_footprint"/>
@@ -14,5 +14,5 @@
       <origin xyz="-0 0 0.2465" rpy="0 0 ${-M_PI*0.5}"/>
       <geometry>
-        <mesh filename="package://mpc_model_description/meshes/body.STL"/>
+        <mesh filename="package://mpc_ros_description/meshes/body.STL"/>
       </geometry>
       <material name="light_black"/>
@@ -37,5 +37,5 @@
       <origin xyz="-0 0 0.2465" rpy="0 0 ${-M_PI*0.5}"/>
       <geometry>
-        <mesh filename="package://mpc_model_description/meshes/base_plate.STL" />
+        <mesh filename="package://mpc_ros_description/meshes/base_plate.STL" />
       </geometry>
       <material
@@ -70,5 +70,5 @@
       <origin xyz="0 0 0" rpy="${-M_PI*0.5} 0 0"/>
       <geometry>
-        <mesh filename="package://mpc_model_description/meshes/left_wheel.STL"/>
+        <mesh filename="package://mpc_ros_description/meshes/left_wheel.STL"/>
       </geometry>
       <material
@@ -102,5 +102,5 @@
       <origin xyz="0 0 -0.025" rpy="${-M_PI*0.5} 0 0"/>
       <geometry>
-        <mesh filename="package://mpc_model_description/meshes/right_wheel.STL"/>
+        <mesh filename="package://mpc_ros_description/meshes/right_wheel.STL"/>
       </geometry>
       <material
@@ -202,5 +202,5 @@
       <origin xyz="0 0 0" rpy="0 0 0"/>
       <geometry>
-        <mesh filename="package://mpc_model_description/meshes/lidar.STL" />
+        <mesh filename="package://mpc_ros_description/meshes/lidar.STL" />
       </geometry>
       <material

File: mpc_ros_description/urdf/holonomic/holonomic.urdf.xacro (robot description, xacro)
@@ -1,6 +1,6 @@
 <?xml version="1.0" ?>
 <robot name="holonomic_bot" xmlns:xacro="http://ros.org/wiki/xacro">
-  <xacro:include filename="$(find mpc_model_description)/urdf/common/common_properties.xacro"/>
-  <xacro:include filename="$(find mpc_model_description)/urdf/holonomic/holonomic.gazebo.xacro"/>
+  <xacro:include filename="$(find mpc_ros_description)/urdf/common/common_properties.xacro"/>
+  <xacro:include filename="$(find mpc_ros_description)/urdf/holonomic/holonomic.gazebo.xacro"/>
   <link name="base_footprint"/>
   <joint name="base_joint" type="fixed">
@@ -88,5 +88,5 @@
       <geometry>
         <mesh
-          filename="package://mpc_model_description/meshes/lidar.STL" />
+          filename="package://mpc_ros_description/meshes/lidar.STL" />
       </geometry>
       <material
@@ -102,5 +102,5 @@
       <geometry>
         <mesh
-          filename="package://mpc_model_description/meshes/lidar.STL" />
+          filename="package://mpc_ros_description/meshes/lidar.STL" />
       </geometry>
     </collision>
